File: esp07_12_shift_inout.brd (EAGLE design)
At the start: 100 x 45 mm, 47 parts, among them IC1 74HCT595D, IC2 74HCT595D, IC3 74HC165D, IC4 74HC165D

Commit message: Another approximation
Parts:
- JP11, JP12: value M02PTH3 -> (none); device SparkFun-Connectors:1X02_LONGPADS -> SparkFun-Connectors:1X02
- JP7: value M02PTH3 -> (none)
- moved R20 21.8 mm to (35.6, 42.5)
- moved R19 19.3 mm to (30.5, 42.5)
- moved JP10 12.7 mm to (11.4, 12.7), turned to 90 degrees
- moved R21 7.73 mm to (45.7, 40.6), turned to 270 degrees
- moved JP12 7.67 mm to (13.3, 8.26)
- moved JP11 7.24 mm to (13.3, 5.71)
- moved JP7 7.10 mm to (13.3, 2.54)
- moved D1 4.58 mm to (19.1, 5.08), turned to 90 degrees
- moved SJ1 3.86 mm to (40.0, 14.0)
- moved R17 3.18 mm to (26.0, 15.2)
- moved R22 2.62 mm to (32.4, 15.2)
- moved JP9 2.54 mm to (11.4, 43.2), turned to 270 degrees
- moved R18 2.54 mm to (29.2, 15.2)
- moved SJ2 2.29 mm to (91.4, 22.2), turned to 90 degrees
- moved U$1 1.27 mm to (41.9, 36.8)
Routing:
- net GND: track 150.7 -> 328.2 mm, vias 5 -> 9
- net VCC: track 171.1 -> 318.1 mm, vias 7 -> 8
- net GPIO15: track 0.00 -> 51.0 mm, vias 0 -> 2
- net OUT_LATCH: track 108.7 -> 149.0 mm, vias 0 -> 2
- net IN_LATCH: track 52.8 -> 91.6 mm, vias 3 -> 4
- net SCK: track 86.0 -> 122.5 mm, vias 5 -> 7
- net GPIO16: track 0.00 -> 31.6 mm, vias 0 -> 2
- net GPIO0: track 0.00 -> 30.9 mm
- net GPIO2: track 0.00 -> 30.5 mm, vias 0 -> 2
- net CH_PD: track 0.00 -> 26.8 mm
- net +12V: track 0.00 -> 23.9 mm
- net RXD: track 0.00 -> 21.3 mm
- net TXD: track 0.00 -> 17.2 mm
- net MISO: track 17.1 -> 33.6 mm
- net MOSI: track 15.0 -> 29.2 mm
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- added copper zone on layer 1, net GND
- added copper zone on layer 16, net GND
- added copper zone on layer 1, net VCC
